Commit message: Imported upstream version '2.5.9' of 'upstream'

File: moveit_planners/test_configs/prbt_support/urdf/prbt.ros2_control.xacro (robot description, xacro)
@@ -19,13 +19,7 @@
 					<param name="max">3.15</param>
 				</command_interface>
-				<state_interface name="position">
-					<param name="initial_value">0.0</param>
-				</state_interface>
-				<state_interface name="velocity">
-					<param name="initial_value">0.0</param>
-				</state_interface>
-				<state_interface name="effort">
-					<param name="initial_value">0.0</param>
-				</state_interface>
+				<state_interface name="position"/>
+				<state_interface name="velocity"/>
+				<state_interface name="effort"/>
 				<param name="initial_position">${initial_positions['joint_1']}</param>  <!-- initial position for the FakeSystem -->
 			</joint>
@@ -39,13 +33,7 @@
 					<param name="max">3.15</param>
 				</command_interface>
-				<state_interface name="position">
-					<param name="initial_value">0.0</param>
-				</state_interface>
-				<state_interface name="velocity">
-					<param name="initial_value">0.0</param>
-				</state_interface>
-				<state_interface name="effort">
-					<param name="initial_value">0.0</param>
-				</state_interface>
+				<state_interface name="position"/>
+				<state_interface name="velocity"/>
+				<state_interface name="effort"/>
 				<param name="initial_position">${initial_positions['joint_2']}</param>  <!-- initial position for the FakeSystem -->
 			</joint>
@@ -59,13 +47,7 @@
 					<param name="max">3.15</param>
 				</command_interface>
-				<state_interface name="position">
-					<param name="initial_value">0.0</param>
-				</state_interface>
-				<state_interface name="velocity">
-					<param name="initial_value">0.0</param>
-				</state_interface>
-				<state_interface name="effort">
-					<param name="initial_value">0.0</param>
-				</state_interface>
+				<state_interface name="position"/>
+				<state_interface name="velocity"/>
+				<state_interface name="effort"/>
 				<param name="initial_position">${initial_positions['joint_3']}</param>  <!-- initial position for the FakeSystem -->
 			</joint>
@@ -79,13 +61,7 @@
 					<param name="max">3.15</param>
 				</command_interface>
-				<state_interface name="position">
-					<param name="initial_value">0.0</param>
-				</state_interface>
-				<state_interface name="velocity">
-					<param name="initial_value">0.0</param>
-				</state_interface>
-				<state_interface name="effort">
-					<param name="initial_value">0.0</param>
-				</state_interface>
+				<state_interface name="position"/>
+				<state_interface name="velocity"/>
+				<state_interface name="effort"/>
 				<param name="initial_position">${initial_positions['joint_4']}</param>  <!-- initial position for the FakeSystem -->
 			</joint>
@@ -99,13 +75,7 @@
 					<param name="max">3.15</param>
 				</command_interface>
-				<state_interface name="position">
-					<param name="initial_value">0.0</param>
-				</state_interface>
-				<state_interface name="velocity">
-					<param name="initial_value">0.0</param>
-				</state_interface>
-				<state_interface name="effort">
-					<param name="initial_value">0.0</param>
-				</state_interface>
+				<state_interface name="position"/>
+				<state_interface name="velocity"/>
+				<state_interface name="effort"/>
 				<param name="initial_position">${initial_positions['joint_5']}</param>  <!-- initial position for the FakeSystem -->
 			</joint>
@@ -119,13 +89,7 @@
 					<param name="max">3.15</param>
 				</command_interface>
-				<state_interface name="position">
-					<param name="initial_value">0.0</param>
-				</state_interface>
-				<state_interface name="velocity">
-					<param name="initial_value">0.0</param>
-				</state_interface>
-				<state_interface name="effort">
-					<param name="initial_value">0.0</param>
-				</state_interface>
+				<state_interface name="position"/>
+				<state_interface name="velocity"/>
+				<state_interface name="effort"/>
 				<param name="initial_position">${initial_positions['joint_6']}</param>  <!-- initial position for the FakeSystem -->
 			</joint>

File: moveit_setup_assistant/moveit_setup_controllers/templates/config/ros2_control.xacro (robot description, xacro)
@@ -2,5 +2,5 @@
 <robot xmlns:xacro="http://www.ros.org/wiki/xacro">
     <xacro:macro name="[ROBOT_NAME]_ros2_control" params="name initial_positions_file">
-        <xacro:property name="initial_positions" value="${xacro.load_yaml(initial_positions_file)['initial_positions']}"/>
+        <xacro:property name="initial_positions" value="${load_yaml(initial_positions_file)['initial_positions']}"/>
         <ros2_control name="${name}" type="system">
             <hardware>
